File: Line_Follower/Line_Follower.kicad_sch (KiCad schematic)
At the start: 25 parts, among them J1 Battery terminal, J10 Motor_B, J11 8-Channel IR Array, J8 I2C (OLED), J9 Motor_A, SW1 Slide Switch, SW3 Mode, SW6 Calibration, U1 ESP32-DEVKITC, U2 LM2596 Buck Converter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

Commit message: Schematic edited
Parts:
- removed J8: I2C (OLED), Connector_PinSocket_2.54mm:PinSocket_1x04_P2.54mm_Vertical, symbol Connector:Conn_01x04_Socket
Connections:
- net SCL: no longer names the net of U1.29 (IO5)
- net SDA: no longer names the net of U1.26 (IO4)
- no-connect marks 16 -> 18
Other:
- note removed: "I2C"
- moved on the sheet: J10, J9, R13, R14, SW3, SW6

Commit message: Net classes assigned
Parts:
- U3: footprint ROB-14450:MODULE_ROB-14450 -> TB6612FNG:TB6612FNG_Driver
Changed lines of the file:
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@@
 			)
 		)
-		(property "Footprint" "ROB-14450:MODULE_ROB-14450"
+		(property "Footprint" "TB6612FNG:TB6612FNG_Driver"
 			(at 50.8 121.92 0)
 			(effects

Commit message: Footprint added, PCB aligned
Parts:
- TP1: value TestPoint -> TP_VBAT
- TP3: value TestPoint -> TP_3V3
- TP4: value TestPoint -> TP_GND
- U3: Availability In Stock -> (none); Check_prices https://www.snapeda.com/parts/ROB-14450/SparkFun/view-part/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 -> (none); Description_1 TB6612FNG - Motor Controller/Driver Power Management Evalua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 -> (none); MANUFACTURER Sparkfun Electronics -> (none); MF SparkFun Electronics -> (none); MP ROB-14450 -> (none); PARTREV 11-13-17 -> (none); Package None -> (none); Price None -> (none); Purchase-URL https://www.snapeda.com/api/url_track_click_mouser/?unipart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 -> (none); STANDARD Manufacturer Recommendation -> (none); SnapEDA_Link https://www.snapeda.com/parts/ROB-14450/SparkFun/view-part/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 -> (none)
Connections:
- net VBAT+: no longer U2.1 (IN+)
- net VBAT_IN+: now reaches J1.1 (Pin_1), SW1.2 (B)
- net VBAT_IN+: now also U2.1 (IN+)

Commit message: PCB updated
Parts:
- removed TP3: TP_3V3, TestPoint:TestPoint_2Pads_Pitch5.08mm_Drill1.3mm, symbol Connector:TestPoint
- TP1: footprint TestPoint:TestPoint_2Pads_Pitch5.08mm_Drill1.3mm -> TestPoint:TestPoint_Pad_2.0x2.0mm
- TP2: renamed from TP4; footprint TestPoint:TestPoint_2Pads_Pitch5.08mm_Drill1.3mm -> TestPoint:TestPoint_Pad_2.0x2.0mm
Changed lines of the file:
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@@
 	(wire
 		(pts
-			(xy 101.6 48.26) (xy 101.6 43.18)
-		)
-		(stroke
-			(width 0)
-			(type default)
-		)
-	)
-	(wire
-		(pts
 			(xy 125.73 78.74) (xy 125.73 72.39)
 		)
@@
 	)
 	(symbol
-		(lib_id "Connector:TestPoint")
-		(at 101.6 48.26 270)
-		(unit 1)
-		(exclude_from_sim no)
-		(in_bom yes)
-		(on_board yes)
-		(dnp no)
-		(fields_autoplaced yes)
-		(property "Reference" "TP3"
-			(at 106.68 46.9899 90)
-			(effects
-				(font
-					(size 1.27 1.27)
-				)
-				(justify left)
-			)
-		)
-		(property "Value" "TP_3V3"
-			(at 106.68 49.5299 90)
-			(effects
-				(font
-					(size 1.27 1.27)
-				)
-				(justify left)
-			)
-		)
-		(property "Footprint" "TestPoint:TestPoint_2Pads_Pitch5.08mm_Drill1.3mm"
-			(at 101.6 53.34 0)
-			(effects
-				(font
-					(size 1.27 1.27)
-				)
-				(hide yes)
-			)
-		)
-		(property "Datasheet" "~"
-			(at 101.6 53.34 0)
-			(effects
-				(font
-					(size 1.27 1.27)
-				)
-				(hide yes)
-			)
-		)
-		(property "Description" "test point"
-			(at 101.6 48.26 0)
-			(effects
-				(font
-					(size 1.27 1.27)
-				)
-				(hide yes)
-			)
-		)
-		(pin "1"
-		)
-		(instances
-			(project "Line_Follower"
-				(path "/defca6a9-24dc-49d0-b78f-524feb7c47ac"
-					(reference "TP3")
-					(unit 1)
-				)
-			)
-		)
-	)
-	(symbol
 		(lib_id "Switch:SW_Push")
 		(at 236.22 100.33 0)
@@
 		(dnp no)
 		(fields_autoplaced yes)
-		(property "Reference" "TP4"
+		(property "Reference" "TP2"
 			(at 25.908 62.23 90)
 			(effects
@@
 			)
 		)
-		(property "Footprint" "TestPoint:TestPoint_2Pads_Pitch5.08mm_Drill1.3mm"
+		(property "Footprint" "TestPoint:TestPoint_Pad_2.0x2.0mm"
 			(at 29.21 62.23 0)
 			(effects
@@
 			(project "Line_Follower"
 				(path "/defca6a9-24dc-49d0-b78f-524feb7c47ac"
-					(reference "TP4")
+					(reference "TP2")
 					(unit 1)
 				)
@@
 			)
 		)
-		(property "Footprint" "TestPoint:TestPoint_2Pads_Pitch5.08mm_Drill1.3mm"
+		(property "Footprint" "TestPoint:TestPoint_Pad_2.0x2.0mm"
 			(at 38.1 38.1 0)
 			(effects

Commit message: PCB edited
Parts:
- removed FID1, FID2, FID3: Fiducial, Fiducial:Fiducial_0.75mm_Mask1.5mm, symbol Mechanical:Fiducial
Other:
- note removed: "FIDUCIAL"
Changed lines of the file:
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@@
 	)
 	(rectangle
-		(start 257.81 20.32)
-		(end 276.86 69.85)
-		(stroke
-			(width 0)
-			(type dash_dot_dot)
-		)
-		(fill
-			(type none)
-		)
-	)
-	(rectangle
 		(start 172.72 100.33)
 		(end 212.09 125.73)
@@
 		)
 	)
-	(text "FIDUCIAL"
-		(exclude_from_sim no)
-		(at 266.954 24.892 0)
-		(effects
-			(font
-				(size 2.032 2.032)
-				(thickness 0.762)
-				(bold yes)
-			)
-		)
-	)
 	(text "MOTOR TERMINALS"
 		(exclude_from_sim no)
@@
 	)
 	(symbol
-		(lib_id "Mechanical:Fiducial")
-		(at 262.89 30.48 0)
-		(unit 1)
-		(exclude_from_sim no)
-		(in_bom no)
-		(on_board yes)
-		(dnp no)
-		(fields_autoplaced yes)
-		(property "Reference" "FID1"
-			(at 265.43 29.2099 0)
-			(effects
-				(font
-					(size 1.27 1.27)
-				)
-				(justify left)
-			)
-		)
-		(property "Value" "Fiducial"
-			(at 265.43 31.7499 0)
-			(effects
-				(font
-					(size 1.27 1.27)
-				)
-				(justify left)
-			)
-		)
-		(property "Footprint" "Fiducial:Fiducial_0.75mm_Mask1.5mm"
-			(at 262.89 30.48 0)
-			(effects
-				(font
-					(size 1.27 1.27)
-				)
-				(hide yes)
-			)
-		)
-		(property "Datasheet" "~"
-			(at 262.89 30.48 0)
-			(effects
-				(font
-					(size 1.27 1.27)
-				)
-				(hide yes)
-			)
-		)
-		(property "Description" "Fiducial Marker"
-			(at 262.89 30.48 0)
-			(effects
-				(font
-					(size 1.27 1.27)
-				)
-				(hide yes)
-			)
-		)
-		(instances
-			(project "Line_Follower"
-				(path "/defca6a9-24dc-49d0-b78f-524feb7c47ac"
-					(reference "FID1")
-					(unit 1)
-				)
-			)
-		)
-	)
-	(symbol
 		(lib_id "Switch:SW_SPDT")
 		(at 44.45 52.07 90)
@@
 	)
 	(symbol
-		(lib_id "Mechanical:Fiducial")
-		(at 262.89 38.1 0)
-		(unit 1)
-		(exclude_from_sim no)
-		(in_bom no)
-		(on_board yes)
-		(dnp no)
-		(fields_autoplaced yes)
-		(property "Reference" "FID2"
-			(at 265.43 36.8299 0)
-			(effects
-				(font
-					(size 1.27 1.27)
-				)
-				(justify left)
-			)
-		)
-		(property "Value" "Fiducial"
-			(at 265.43 39.3699 0)
-			(effects
-				(font
-					(size 1.27 1.27)
-				)
-				(justify left)
-			)
-		)
-		(property "Footprint" "Fiducial:Fiducial_0.75mm_Mask1.5mm"
-			(at 262.89 38.1 0)
-			(effects
-				(font
-					(size 1.27 1.27)
-				)
-				(hide yes)
-			)
-		)
-		(property "Datasheet" "~"
-			(at 262.89 38.1 0)
-			(effects
-				(font
-					(size 1.27 1.27)
-				)
-				(hide yes)
-			)
-		)
-		(property "Description" "Fiducial Marker"
-			(at 262.89 38.1 0)
-			(effects
-				(font
-					(size 1.27 1.27)
-				)
-				(hide yes)
-			)
-		)
-		(instances
-			(project "Line_Follower"
-				(path "/defca6a9-24dc-49d0-b78f-524feb7c47ac"
-					(reference "FID2")
-					(unit 1)
-				)
-			)
-		)
-	)
-	(symbol
 		(lib_id "power:GND")
 		(at 73.66 135.89 0)
@@
 					(unit 1)
 				)
-			)
-		)
-	)
-	(symbol
-		(lib_id "Mechanical:Fiducial")
-		(at 262.89 45.72 0)
-		(unit 1)
-		(exclude_from_sim no)
-		(in_bom no)
-		(on_board yes)
-		(dnp no)
-		(fields_autoplaced yes)
-		(property "Reference" "FID3"
-			(at 265.43 44.4499 0)
-			(effects
-				(font
-					(size 1.27 1.27)
-				)
-				(justify left)
-			)
-		)
-		(property "Value" "Fiducial"
-			(at 265.43 46.9899 0)
-			(effects
-				(font
-					(size 1.27 1.27)
-				)
-				(justify left)
-			)
-		)
-		(property "Footprint" "Fiducial:Fiducial_0.75mm_Mask1.5mm"
-			(at 262.89 45.72 0)
-			(effects
-				(font
-					(size 1.27 1.27)
-				)
-				(hide yes)
-			)
-		)
-		(property "Datasheet" "~"
-			(at 262.89 45.72 0)
-			(effects
-				(font
-					(size 1.27 1.27)
-				)
-				(hide yes)
-			)
-		)
-		(property "Description" "Fiducial Marker"
-			(at 262.89 45.72 0)
-			(effects
-				(font
-					(size 1.27 1.27)
-				)
-				(hide yes)
-			)
-		)
-		(instances
-			(project "Line_Follower"
-				(path "/defca6a9-24dc-49d0-b78f-524feb7c47ac"
-					(reference "FID3")
-					(unit 1)
-				)

Commit message: PCB updated
Parts:
- added H1, H2, H3, H4: MountingHole, MountingHole:MountingHole_3.2mm_M3, symbol Mechanical:MountingHole
Other:
- note added: "MOUNTING HOLES"

Commit message: Routing started
Connections:
- net VBAT+: now also U2.1 (IN+)
- net VBAT_IN+: no longer names the net of J1.1 (Pin_1), SW1.2 (B)
- net VBAT_IN+: no longer U2.1 (IN+)
Changed lines of the file:
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@@
-	)
-	(junction
-		(at 44.45 59.69)
-		(diameter 0)
-		(color 0 0 0 0)
 	)
 	(junction
@@
 	(wire
 		(pts
-			(xy 44.45 60.96) (xy 44.45 59.69)
-		)
-		(stroke
-			(width 0)
-			(type default)
-		)
-	)
-	(wire
-		(pts
 			(xy 135.89 52.07) (xy 139.7 52.07)
 		)
@@
 	(wire
 		(pts
-			(xy 44.45 59.69) (xy 49.53 59.69)
-		)
-		(stroke
-			(width 0)
-			(type default)
-		)
-	)
-	(wire
-		(pts
 			(xy 95.25 111.76) (xy 99.06 111.76)
 		)
@@
 	(wire
 		(pts
-			(xy 44.45 59.69) (xy 44.45 57.15)
+			(xy 44.45 57.15) (xy 44.45 60.96)
 		)
 		(stroke
@@
 		)
 	)
-	(global_label "VBAT_IN+"
+	(global_label "VBAT+"
 		(shape input)
 		(at 76.2 43.18 90)
@@
 		)
 		(property "Intersheetrefs" "${INTERSHEET_REFS}"
-			(at 76.2 31.3047 90)
+			(at 76.2 34.2076 90)
 			(effects
 				(font
@@
 				)
 				(justify right)
-				(hide yes)
-			)
-		)
-	)
-	(global_label "VBAT_IN+"
-		(shape input)
-		(at 49.53 59.69 0)
-		(fields_autoplaced yes)
-		(effects
-			(font
-				(size 1.27 1.27)
-			)
-			(justify left)
-		)
-		(property "Intersheetrefs" "${INTERSHEET_REFS}"
-			(at 61.4053 59.69 0)
-			(effects
-				(font
-					(size 1.27 1.27)
-				)
-				(justify left)
 				(hide yes)
 			)
@@
 			)
 		)
+	)
+	(netclass_flag ""
+		(length 2.54)
+		(shape round)
+		(at 44.45 60.96 270)
+		(fields_autoplaced yes)
+		(effects
+			(font
+				(size 1.27 1.27)
+			)
+			(justify right bottom)
+		)
+		(property "Netclass" "VBAT"
+			(at 46.99 60.2615 90)
+			(effects
+				(font
+					(size 1.27 1.27)
+				)
+				(justify left)
+				(hide yes)
+			)
+		)
+		(property "Component Class" ""
+			(at -71.12 6.35 0)
+			(effects
+				(font
+					(size 1.27 1.27)
+					(italic yes)
+				)
+			)
+		)

Commit message: Routing done
Parts:
- C5, C8: footprint (none) -> Capacitors:C320C
- C6, C7: footprint (none) -> Capacitors:CAPPRD750W80D1600H2500
Changed lines of the file:
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@@
 			)
 		)
-		(property "Footprint" ""
+		(property "Footprint" "Capacitors:CAPPRD750W80D1600H2500"
 			(at 86.0552 134.62 0)
 			(effects
@@
 			)
 		)
-		(property "Footprint" ""
+		(property "Footprint" "Capacitors:C320C"
 			(at 96.2152 110.49 0)
 			(effects
@@
 			)
 		)
-		(property "Footprint" ""
+		(property "Footprint" "Capacitors:C320C"
 			(at 93.6752 134.62 0)
 			(effects
@@
 			)
 		)
-		(property "Footprint" ""
+		(property "Footprint" "Capacitors:CAPPRD750W80D1600H2500"
 			(at 103.8352 110.49 0)
 			(effects
