File: Line_Follower/Line_Follower.kicad_pcb (KiCad board)
At the start: 2 copper layers, 95.5 x 93.5 mm, 20 parts, among them J1 Battery terminal, J10 Motor_B, J11 8-Channel IR Array, J9 Motor_A, SW1 Slide Switch, SW3 Mode, SW6 Calibration, U1 ESP32-DEVKITC, U2 LM2596 Buck Converter, U3 TB6612FNG_MD

Commit message: PCB edited
Parts:
- moved H1 18.8 mm to (104.2, 35.8)
- moved H2 18.8 mm to (188.2, 35.8)
- moved J10 6.52 mm to (186.3, 49.0)
- moved J9 6.35 mm to (106.2, 43.8)
- moved R13 6.21 mm to (134.5, 46.8)
- moved R14 6.21 mm to (120.2, 46.8)
- moved R2 3.06 mm to (164.8, 48.8), turned to 180 degrees
- moved U3 2.76 mm to (122.0, 66.2)
- moved SW1 2.51 mm to (173.7, 34.0)
- moved D2 2.50 mm to (174.8, 46.5)
- moved H3 2.24 mm to (115.2, 117.8)
- moved H4 2.24 mm to (177.2, 117.8)
- moved U2 1.71 mm to (136.8, 76.4)
- moved U1 1.32 mm to (148.8, 94.7)
- moved J1 0.46 mm to (158.8, 38.0)
Routing:
- net 3V3: track 0.00 -> 0.85 mm
Other:
- board text added: "IN+"
- board text added: "IN-"
- board text added: "OUT+"
- board text added: "OUT-"
Changed lines of the file:
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@@
 	(footprint "Resistor_THT:R_Axial_DIN0207_L6.3mm_D2.5mm_P10.16mm_Horizontal"
 		(layer "F.Cu")
-		(at 126.38 45.7375)
+		(at 120.25 46.75)
 		(descr "Resistor, Axial_DIN0207 series, Axial, Horizontal, pin pitch=10.16mm, 0.25W = 1/4W, length*diameter=6.3*2.5mm^2, http://cdn-reichelt.de/documents/datenblatt/B400/1_4W%23YAG.pdf")
 		(tags "Resistor Axial_DIN0207 series Axial Horizontal pin pitch 10.16mm 0.25W = 1/4W length 6.3mm diameter 2.5mm")
@@
 	(footprint "Button_Switch_THT:SW_Slide-03_Wuerth-WS-SLTV_10x2.5x6.4_P2.54mm"
 		(layer "F.Cu")
-		(at 171.21 34.2375)
+		(at 173.71 34)
 		(descr "Wuerth, WS-SLTV, 450301014042, https://www.we-online.com/components/products/datasheet/450301014042.pdf")
 		(tags "switch single-pole opposite-side-connection double-throw SPDT würth wurth")
@@
 	(footprint "Screw Terminal:CUI_TB007-508-02BE"
 		(layer "F.Cu")
-		(at 185.7625 42.54 90)
+		(at 186.2625 49.04 90)
 		(property "Reference" "J10"
-			(at -4.46 -0.0125 180)
+			(at 9.29 -4.2625 0)
 			(layer "F.SilkS")
 			(effects
@@
 	(footprint "MountingHole:MountingHole_3.2mm_M3"
 		(layer "F.Cu")
-		(at 176.25 115.75)
+		(at 177.25 117.75)
 		(descr "Mounting Hole 3.2mm, M3, no annular, generated by kicad-footprint-generator mountinghole.py")
 		(tags "mountinghole M3")
@@
 		)
 		(property "Value" "MountingHole"
-			(at 0 4.15 0)
+			(at -5 -0.5 90)
 			(layer "F.Fab")
 			(effects
@@
 	(footprint "LED_THT:LED_D5.0mm"
 		(layer "F.Cu")
-		(at 176.25 44.5 180)
+		(at 174.75 46.5 180)
 		(descr "LED, diameter 5.0mm, 2 pins, http://cdn-reichelt.de/documents/datenblatt/A500/LL-504BC2E-009.pdf, generated by kicad-footprint-generator")
 		(tags "LED")
@@
 	(footprint "Screw Terminal:CUI_TB007-508-02BE"
 		(layer "F.Cu")
-		(at 106.7375 37.42 -90)
+		(at 106.25 43.75 -90)
 		(property "Reference" "J9"
-			(at 9.58 -0.2625 0)
+			(at -3.75 -3.25 0)
 			(layer "F.SilkS")
 			(effects
@@
 	(footprint "Buck_Converter:LM2596_Buck_Module"
 		(layer "F.Cu")
-		(at 137.2616 74.7402)
+		(at 136.85 76.4)
 		(property "Reference" "U2"
 			(at 21.5 -12 0)
@@
 	(footprint "MountingHole:MountingHole_3.2mm_M3"
 		(layer "F.Cu")
-		(at 116.25 115.75)
+		(at 115.25 117.75)
 		(descr "Mounting Hole 3.2mm, M3, no annular, generated by kicad-footprint-generator mountinghole.py")
 		(tags "mountinghole M3")
@@
 		)
 		(property "Value" "MountingHole"
-			(at 0 4.15 0)
+			(at 4.75 -0.75 90)
 			(layer "F.Fab")
 			(effects
@@
 	(footprint "ESP-WROOM:MODULE_ESP32-DEVKITC"
 		(layer "F.Cu")
-		(at 148.37 93.45 90)
+		(at 148.79 94.7 90)
 		(property "Reference" "U1"
 			(at -10.795 -31.75 90)
@@
 	(footprint "Resistor_THT:R_Axial_DIN0207_L6.3mm_D2.5mm_P10.16mm_Horizontal"
 		(layer "F.Cu")
-		(at 140.63 45.7375)
+		(at 134.5 46.75)
 		(descr "Resistor, Axial_DIN0207 series, Axial, Horizontal, pin pitch=10.16mm, 0.25W = 1/4W, length*diameter=6.3*2.5mm^2, http://cdn-reichelt.de/documents/datenblatt/B400/1_4W%23YAG.pdf")
 		(tags "Resistor Axial_DIN0207 series Axial Horizontal pin pitch 10.16mm 0.25W = 1/4W length 6.3mm diameter 2.5mm")
@@
 	(footprint "MountingHole:MountingHole_3.2mm_M3"
 		(layer "F.Cu")
-		(at 187.5 54.5)
+		(at 188.25 35.75)
 		(descr "Mounting Hole 3.2mm, M3, no annular, generated by kicad-footprint-generator mountinghole.py")
 		(tags "mountinghole M3")
 		(property "Reference" "H2"
-			(at -1.75 6.75 0)
+			(at -4.5 -4.5 0)
 			(layer "F.SilkS")
 			(effects
@@
 		)
 		(property "Value" "MountingHole"
-			(at 0 4.15 0)
+			(at -3 -4.5 0)
 			(layer "F.Fab")
 			(effects
@@
 	(footprint "MountingHole:MountingHole_3.2mm_M3"
 		(layer "F.Cu")
-		(at 105 54.5)
+		(at 104.25 35.75)
 		(descr "Mounting Hole 3.2mm, M3, no annular, generated by kicad-footprint-generator mountinghole.py")
 		(tags "mountinghole M3")
 		(property "Reference" "H1"
-			(at 1 6.5 0)
+			(at 2.75 -4.25 0)
 			(layer "F.SilkS")
 			(effects
@@
 		)
 		(property "Value" "MountingHole"
-			(at 0 4.15 0)
+			(at 1.25 -4.25 0)
 			(layer "F.Fab")
 			(effects
@@
 			(at 0.25 -4.05 180)
 			(layer "F.SilkS")
+			(hide yes)
 			(effects
 				(font
@@
 	(footprint "TB6612FNG:TB6612FNG_Driver"
 		(layer "F.Cu")
-		(at 122.63 63.56)
+		(at 122 66.25)
 		(property "Reference" "U3"
 			(at -5.5332 -11.6132 0)
@@
 	(footprint "Resistor_THT:R_Axial_DIN0207_L6.3mm_D2.5mm_P10.16mm_Horizontal"
 		(layer "F.Cu")
-		(at 167.75 49.33 90)
+		(at 164.75 48.75 180)
 		(descr "Resistor, Axial_DIN0207 series, Axial, Horizontal, pin pitch=10.16mm, 0.25W = 1/4W, length*diameter=6.3*2.5mm^2, http://cdn-reichelt.de/documents/datenblatt/B400/1_4W%23YAG.pdf")
 		(tags "Resistor Axial_DIN0207 series Axial Horizontal pin pitch 10.16mm 0.25W = 1/4W length 6.3mm diameter 2.5mm")
 		(property "Reference" "R2"
-			(at 5.08 2.5 90)
+			(at 2 2.5 0)
 			(layer "F.SilkS")
 			(effects
@@
 		)
 		(property "Value" "220"
-			(at 5.08 2.37 90)
+			(at 5.08 2.37 0)
 			(layer "F.Fab")
 			(effects
@@
 		)
 		(property "Datasheet" "~"
-			(at 0 0 90)
+			(at 0 0 0)
 			(layer "F.Fab")
 			(hide yes)
@@
 		)
 		(property "Description" "Resistor"
-			(at 0 0 90)
+			(at 0 0 0)
 			(layer "F.Fab")
 			(hide yes)
@@
 		)
 		(fp_text user "${REFERENCE}"
-			(at 5.08 0 90)
+			(at 5.08 0 0)
 			(layer "F.Fab")
 			(effects
@@
 		)
 		(pad "1" thru_hole circle
-			(at 0 0 90)
+			(at 0 0 180)
 			(size 1.6 1.6)
 			(drill 0.8)
@@
 		)
 		(pad "2" thru_hole circle
-			(at 10.16 0 90)
+			(at 10.16 0 180)
 			(size 1.6 1.6)
 			(drill 0.8)
@@
 	(footprint "Screw Terminal:CUI_TB007-508-02BE"
 		(layer "F.Cu")
-		(at 158.33 38 180)
+		(at 158.79 37.9875 180)
 		(property "Reference" "J1"
 			(at 0.905 -7.239 0)
@@
 	)
 	(gr_text "10K"
-		(at 131.54 48.9875 0)
+		(at 125.41 50 0)
 		(layer "F.SilkS")
 		(effects
@@
 		)
 	)
+	(gr_text "IN+"
+		(at 137.25 54.5 0)
+		(layer "F.SilkS")
+		(effects
+			(font
+				(size 1 1)
+				(thickness 0.1875)
+			)
+			(justify left bottom)
+		)
+	)
 	(gr_text "+"
-		(at 158.33 32.25 0)
+		(at 158.79 32.1875 0)
 		(layer "F.SilkS")
 		(effects
@@
 	)
 	(gr_text "10K"
-		(at 146.04 48.9875 0)
+		(at 139.91 50 0)
 		(layer "F.SilkS")
 		(effects
@@
 		)
 	)
+	(gr_text "IN-"
+		(at 137.25 78.5 0)
+		(layer "F.SilkS")
+		(effects
+			(font
+				(size 1 1)
+				(thickness 0.1875)
+			)
+			(justify left bottom)
+		)
+	)
 	(gr_text "IR2"
 		(at 138.25 120.25 90)
@@
 	)
 	(gr_text "+LED-"
-		(at 172.5 50.5 0)
+		(at 171 51.75 0)
 		(layer "F.SilkS")
 		(effects
@@
 	)
 	(gr_text "Power"
-		(at 173.67 30.9875 180)
+		(at 175.5 30.75 180)
 		(layer "F.SilkS")
 		(effects
@@
 		)
 	)
+	(gr_text "OUT-"
+		(at 177 78.75 0)
+		(layer "F.SilkS")
+		(effects
+			(font
+				(size 1 1)
+				(thickness 0.1875)
+			)
+			(justify left bottom)
+		)
+	)
 	(gr_text "MB"
-		(at 187 32.75 180)
+		(at 193.25 47.25 90)
 		(layer "F.SilkS")
 		(effects
@@
 	)
 	(gr_text "MA"
-		(at 108 32.75 180)
+		(at 99.25 45.75 270)
 		(layer "F.SilkS")
 		(effects
@@
 		)
 	)
+	(gr_text "OUT+"
+		(at 176.25 54.5 0)
+		(layer "F.SilkS")
+		(effects
+			(font
+				(size 1 1)
+				(thickness 0.1875)
+			)
+			(justify left bottom)
+		)
+	)
 	(gr_text "220"
-		(at 164.75 50 90)
+		(at 158.25 52.25 0)
 		(layer "F.SilkS")
 		(effects
@@
 	)
 	(gr_text "-"
-		(at 152.58 32.25 0)
+		(at 153 32.25 0)
 		(layer "F.SilkS")
 		(effects
@@
 		)
 	)
+	(segment
+		(start 178.25 57)
+		(end 177.4992 57)
+		(width 0.5)
+		(layer "F.Cu")
+		(net 16)
+	)
+	(segment
+		(start 120.3192 46.8192)
+		(end 120.25 46.75)
+		(width 0.5)
+		(layer "B.Cu")
+		(net 16)
+	)
 	(group ""

Commit message: Routing started
Parts:
- moved R2 10.2 mm to (154.5, 48.8), turned to 0 degrees
Connections:
- J1 pad 1: VBAT_IN+ -> Net-(J1-Pin_1)
- SW1 pad 2: VBAT_IN+ -> Net-(J1-Pin_1)
- U2 pad 1: VBAT_IN+ -> VBAT+
Routing:
- net GND: track 0.00 -> 185.4 mm
- net 3V3: track 0.85 -> 183.6 mm, vias 0 -> 1
- net VBAT+: track 0.00 -> 109.4 mm, vias 0 -> 1
- net MB1: track 0.00 -> 84.9 mm
- net MB2: track 0.00 -> 82.7 mm
- net PWMB: track 0.00 -> 59.6 mm, vias 0 -> 3
- net PWMA: track 0.00 -> 58.2 mm, vias 0 -> 1
- net MODE: track 0.00 -> 56.2 mm, vias 0 -> 2
- net CAL: track 0.00 -> 51.4 mm, vias 0 -> 2
- net IR8: track 0.00 -> 41.7 mm
- net IR1: track 0.00 -> 35.4 mm
- net AIN2: track 0.00 -> 33.4 mm
- net AIN1: track 0.00 -> 29.8 mm
- net MA1: track 0.00 -> 24.6 mm
- net MA2: track 0.00 -> 22.1 mm
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
Commit message: Routing done
Parts:
- added C5: 100nF, Capacitors:C320C, F.Cu at (113.0, 65.0)
- added C8: 100nF, Capacitors:C320C, F.Cu at (102.0, 59.5)
- moved R2 52.1 mm to (176.8, 95.8), turned to 90 degrees
- moved D2 30.9 mm to (178.0, 77.2)
- moved H4 8.75 mm to (177.5, 109.0)
- moved H3 8.75 mm to (115.2, 109.0)
- moved J11 7.50 mm to (134.8, 107.2)
- moved U1 7.40 mm to (145.2, 88.2)
- moved U3 7.31 mm to (123.5, 59.1)
- moved U2 6.22 mm to (136.0, 70.2)
- moved R14 2.83 mm to (118.9, 44.2)
- moved R13 2.63 mm to (133.7, 44.2)
- moved SW3 1.00 mm to (128.2, 34.3)
- moved SW6 1.00 mm to (139.5, 34.2)
- moved TP1 1.00 mm to (116.0, 35.5)
- moved TP2 1.00 mm to (121.5, 35.3)
- moved J10 0.87 mm to (186.8, 48.3)
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Routing:
- net GND: track 185.4 -> 0.02 mm
- net BIN2: track 0.00 -> 49.1 mm
- net BIN1: track 0.00 -> 47.4 mm
- net VBAT+: track 109.4 -> 134.0 mm, vias 1 -> 0
- net 3V3: track 183.6 -> 207.4 mm, vias 1 -> 0
- net PWMB: track 59.6 -> 41.3 mm, vias 3 -> 0
- net MODE: track 56.2 -> 48.2 mm, vias 2 -> 0
- net IR8: track 41.7 -> 48.1 mm
- net MA2: track 22.1 -> 16.2 mm
- net MA1: track 24.6 -> 19.5 mm
- net MB1: track 84.9 -> 88.3 mm, vias 0 -> 1
- net CAL: track 51.4 -> 54.6 mm
- net AIN2: track 33.4 -> 30.7 mm
- net AIN1: track 29.8 -> 27.1 mm
- net IR6: track 9.97 -> 12.5 mm
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- added copper zone on B.Cu, net GND
- added copper zone on F.Cu, net GND
Other:
- board size 95.5 x 93.5 mm -> 95.5 x 84.7 mm

Commit message: Routing optimised
Parts:
- added G***: LOGO, OP:OP, F.Cu at (120.8, 90.8)
Other:
- board text added: "TracerX"
